File: Hardware/Development/Simulations/adc1_2021-02-04.sch (KiCad schematic (older format))
At the start: 16 parts, among them U1 OPAMP, U2 OPAMP, U3 OPAMP

Commit message: Add files for RevB PCB.
Parts:
- added R10: 500, symbol Device:R
- added R11: 4.5k, symbol Device:R
- added R9: 30k, symbol Device:R
- added V4: pulse(0, 3.3, 1m, 0, 0, 1m), symbol pspice:VSOURCE
- added V5: pulse(0, 3.3, 3m, 0, 0, 1m), symbol pspice:VSOURCE
- U1, U2, U3: Spice_Lib_File /Users/brett/Documents/KiCad/Libraries/Spice Models/LM6211_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 -> C:\\Users\\brett\\Documents\\Kicad\\Libraries\\Spice Models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
Connections:
- net GND: now also R10.2, V4.2 (E2), V5.2 (E2); no longer U1.1 (+)
- net at C1.1, R1.2, R3.2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: now also R9.1
- new net: R10.1, R11.2, U1.1 (+)
- new net: R11.1, V5.1 (E1)
- new net: R9.2, V4.1 (E1)
Changed lines of the file:
@@
 	3450 3150 3400 3150
 Wire Wire Line
-	3400 3150 3400 5000
+	3400 3150 3400 4300
 $Comp
 L power:VDD #PWR010
@@
 F 6 "Y" H 7750 3250 50  0001 C CNN "Spice_Netlist_Enabled"
 F 7 "1 2 4 5 3" H 7750 3250 50  0001 C CNN "Spice_Node_Sequence"
-F 8 "/Users/brett/Documents/KiCad/Libraries/Spice Models/LM6211_PSPICE/LM6211.MOD" H 7750 3250 50  0001 C CNN "Spice_Lib_File"
+F 8 "C:\\Users\\brett\\Documents\\Kicad\\Libraries\\Spice Models\\LM6211_PSPICE\\LM6211.MOD" H 7750 3250 50  0001 C CNN "Spice_Lib_File"
 	1    7750 3250
 	1    0    0    -1
@@
 F 6 "Y" H 5750 3250 50  0001 C CNN "Spice_Netlist_Enabled"
 F 7 "1 2 4 5 3" H 5750 3250 50  0001 C CNN "Spice_Node_Sequence"
-F 8 "/Users/brett/Documents/KiCad/Libraries/Spice Models/LM6211_PSPICE/LM6211.MOD" H 5750 3250 50  0001 C CNN "Spice_Lib_File"
+F 8 "C:\\Users\\brett\\Documents\\Kicad\\Libraries\\Spice Models\\LM6211_PSPICE\\LM6211.MOD" H 5750 3250 50  0001 C CNN "Spice_Lib_File"
 	1    5750 3250
 	1    0    0    -1
@@
 F 6 "Y" H 3750 3250 50  0001 C CNN "Spice_Netlist_Enabled"
 F 7 "1 2 4 5 3" H 3750 3250 50  0001 C CNN "Spice_Node_Sequence"
-F 8 "/Users/brett/Documents/KiCad/Libraries/Spice Models/LM6211_PSPICE/LM6211.MOD" H 3750 3250 50  0001 C CNN "Spice_Lib_File"
+F 8 "C:\\Users\\brett\\Documents\\Kicad\\Libraries\\Spice Models\\LM6211_PSPICE\\LM6211.MOD" H 3750 3250 50  0001 C CNN "Spice_Lib_File"
 	1    3750 3250
 	1    0    0    -1
@@
 	0    1    1    0
 $EndComp
+$Comp
+L pspice:VSOURCE V5
+U 1 1 60DA7C6D
+P 4400 5000
+F 0 "V5" H 4628 5046 50  0000 L CNN
+F 1 "pulse(0, 3.3, 3m, 0, 0, 1m)" H 4628 4955 50  0000 L CNN
+F 2 "" H 4400 5000 50  0001 C CNN
+F 3 "~" H 4400 5000 50  0001 C CNN
+	1    4400 5000
+	1    0    0    -1
+$EndComp
+$Comp
+L pspice:VSOURCE V4
+U 1 1 60DA812D
+P 1000 4250
+F 0 "V4" H 1228 4296 50  0000 L CNN
+F 1 "pulse(0, 3.3, 1m, 0, 0, 1m)" H 1228 4205 50  0000 L CNN
+F 2 "" H 1000 4250 50  0001 C CNN
+F 3 "~" H 1000 4250 50  0001 C CNN
+	1    1000 4250
+	1    0    0    -1
+$EndComp
+$Comp
+L Device:R R9
+U 1 1 60DA8B6D
+P 1250 3350
+F 0 "R9" V 1043 3350 50  0000 C CNN
+F 1 "30k" V 1134 3350 50  0000 C CNN
+F 2 "" V 1180 3350 50  0001 C CNN
+F 3 "~" H 1250 3350 50  0001 C CNN
+	1    1250 3350
+	0    1    1    0
+$EndComp
+Wire Wire Line
+	1100 3350 1000 3350
+Wire Wire Line
+	1000 3350 1000 3950
+Wire Wire Line
+	1000 4550 1000 5000
+Wire Wire Line
+	1000 5000 2250 5000
+Wire Wire Line
+	1400 3350 3000 3350
+Wire Wire Line
+	3400 4950 3400 5000
+Wire Wire Line
+	3750 4300 3400 4300
+Connection ~ 3400 4300
+Wire Wire Line
+	3400 4300 3400 4650
+Wire Wire Line
+	4050 4300 4400 4300
+Wire Wire Line
+	4400 4300 4400 4700
+Wire Wire Line
+	4400 5300 2650 5300
+Wire Wire Line
+	2650 5300 2650 5000
+Wire Wire Line
+	2650 5000 2400 5000
+Connection ~ 2400 5000
+$Comp
+L Device:R R10
+U 1 1 60DADB70
+P 3400 4800
+F 0 "R10" H 3470 4846 50  0000 L CNN
+F 1 "500" H 3470 4755 50  0000 L CNN
+F 2 "" V 3330 4800 50  0001 C CNN
+F 3 "~" H 3400 4800 50  0001 C CNN
+	1    3400 4800
+	1    0    0    -1
+$EndComp
+$Comp
+L Device:R R11
+U 1 1 60DAE3D1
+P 3900 4300
+F 0 "R11" V 3693 4300 50  0000 C CNN
+F 1 "4.5k" V 3784 4300 50  0000 C CNN
+F 2 "" V 3830 4300 50  0001 C CNN
+F 3 "~" H 3900 4300 50  0001 C CNN
+	1    3900 4300
+	0    1    1    0
+$EndComp
