File: Hardware/PCB/SensReadPCB.sch (KiCad schematic (older format))
At the start: 77 parts, among them J1 Conn_02x20_Odd_Even, J2 Barrel_Jack, J3 Screw_Terminal_01x04, J4 Screw_Terminal_01x04, J5 Screw_Terminal_01x03, J6 Conn_02x04_Odd_Even, J7 Conn_01x02_Male, SW1 SW_RESET, SW2 SW_CAL, SW3 SW_TRIG, SW4 SW_AUX, U1 SN74LV1T34DBVR, U2 LM6142AIM, U3 ADP7142AUJZ-R7, U4 AD7724ASTZ, U5 TLE2426xD, U6 LMH6619MA_NOPB

Commit message: Enclosure design added.
Parts:
- U2: symbol Rev2-rescue:LM6142AIM-LM6142AIM -> LM6142AIM:LM6142AIM
Connections:
- wire segments 367 -> 359
Changed lines of the file:
@@
 I_EXC
-Wire Wire Line
-	9800 4400 9800 4500
-Wire Wire Line
-	9800 5300 9800 5400
-Connection ~ 9800 4400
-Connection ~ 9800 4500
-Wire Wire Line
-	9800 4500 9800 4600
-Connection ~ 9800 4600
-Wire Wire Line
-	9800 4600 9800 4700
-Connection ~ 9800 4700
-Wire Wire Line
-	9800 4700 9800 4800
-Connection ~ 9800 5300
-Connection ~ 9800 5400
-Wire Wire Line
-	9800 5400 9800 5500
-Connection ~ 9800 5500
-Wire Wire Line
-	9800 5500 9800 5600
-Connection ~ 9800 5600
-Wire Wire Line
-	9800 5600 9800 5700
-Connection ~ 9800 5700
-Wire Wire Line
-	9800 5700 9800 5800
-Connection ~ 9800 5800
-Wire Wire Line
-	9800 5800 9800 5900
-Connection ~ 9800 6100
 Wire Wire Line
 	4600 5300 4850 5300
@@
 $EndComp
 $Comp
-L Rev2-rescue:LM6142AIM-LM6142AIM U2
+L LM6142AIM:LM6142AIM U2
 U 1 1 61434DFC
 P 3050 4750
@@
 Wire Wire Line
 	4100 5250 4100 5150
-Connection ~ 3750 5150
 $Comp
 L Device:C C2
@@
 Wire Wire Line
 	5300 550  5300 1000
+Wire Wire Line
+	9800 4400 9800 4800
+Wire Wire Line
+	9800 5300 9800 5900
 $EndSCHEMATC
