File: Hardware/PCB/SensReadPCB.sch (KiCad schematic (older format))
At the start: 77 parts, among them J1 Conn_02x20_Odd_Even, J2 Barrel_Jack, J3 Screw_Terminal_01x04, J4 Screw_Terminal_01x04, J5 Screw_Terminal_01x03, J6 Conn_02x04_Odd_Even, J7 Conn_01x02_Male, SW1 SW_RESET, SW2 SW_CAL, SW3 SW_TRIG, SW4 SW_AUX, U1 SN74LV1T34DBVR, U2 LM6142AIM, U3 ADP7142AUJZ-R7, U4 AD7724ASTZ, U5 TLE2426xD, U6 LMH6619MA_NOPB

Commit message: Fixed error in IQ mode (2)
Parts:
- U6: symbol Rev2-rescue:LMH6619MA_NOPB-2021-08-27_19-45-09 -> 2021-09-17_11-40-57:LMH6619MA_NOPB
Changed lines of the file:
@@
 $EndComp
 $Comp
-L Rev2-rescue:LMH6619MA_NOPB-2021-08-27_19-45-09 U6
+L 2021-09-17_11-40-57:LMH6619MA_NOPB U6
 U 1 1 61378695
 P 7650 2300
