File: Hardware/PCB/SensReadPCB.kicad_pcb (KiCad board)
At the start: 2 copper layers, 45.7 x 76.2 mm, 80 parts, among them J1 Conn_02x20_Odd_Even, J2 Barrel_Jack, J3 Screw_Terminal_01x04, J4 Screw_Terminal_01x04, J5 Screw_Terminal_01x03, J6 Conn_02x04_Odd_Even, J7 Conn_01x02_Male, SW1 SW_RESET, SW2 SW_CAL, SW3 SW_TRIG, SW4 SW_AUX, U1 SN74LV1T34DBVR, U2 LM6142AIM, U3 ADP7142AUJZ-R7, U4 AD7724ASTZ, U5 TLE2426xD, U6 LMH6619MA_NOPB

Commit message: Version used for paper
Parts:
- U1: value SN74LV1T34DBVR -> DBV0005A_N
- U4: value AD7724ASTZ -> ST_48_ADI
